File: CAN-BUS_V1.kicad_pcb (KiCad board)
At the start: 2 copper layers, 50 x 36 mm, 45 parts, among them J1 HEADER_4, J2 HEADER_4, J3 HEADER_10, J4 HEADER_10, J5 USB_B_Micro, J6 HEADER_2, J7 HEADER_2, Q1 BC847, Q2 BC847, SW1 SW_Push, U1 DRV8872, U2 esp32-s2-wroom, U3 DRV8872, U4 CH340G, U5 MCP2515-xSO, U6 TJA1050

Commit message: MODIFICACIONES
se modifico sch,pcb  y se elimino un archivo jpg
Connections:
- J3 pad 3: /IO1 -> (no net)
- U1 pad 2: (no net) -> /M1B
- U1 pad 3: (no net) -> /M1A
- U2 pad 15: (no net) -> /M2B
- U2 pad 17: (no net) -> /M2A
- U2 pad 3: /IO0 -> /M1B
- U2 pad 4: /IO1 -> /M1A
- U3 pad 2: (no net) -> /M2B
- U3 pad 3: (no net) -> /M2A
Routing:
- net /M2A: track 0.00 -> 16.6 mm, vias 0 -> 1
- net /M2B: track 0.00 -> 15.3 mm, vias 0 -> 1
- net /M1A: track 0.00 -> 8.42 mm
- net /IO1: track 8.42 -> 0.00 mm
