File: CAN-BUS_V1.sch (KiCad schematic (older format))
At the start: 45 parts, among them J1 HEADER_4, J2 HEADER_4, J3 HEADER_10, J4 HEADER_10, J5 USB_B_Micro, J6 HEADER_2, J7 HEADER_2, Q1 BC847, Q2 BC847, SW1 SW_Push, U1 DRV8872, U2 esp32-s2-wroom, U3 DRV8872, U4 CH340G, U5 MCP2515-xSO, U6 TJA1050

Commit message: MODIFICACIONES
se modifico sch,pcb  y se elimino un archivo jpg
Connections:
- net IO0: no longer U2.3 (IO0)
- net IO1: no longer U2.4 (IO1)
- net IO12: no longer U2.15 (IO12)
- net M1A: now also U2.4 (IO1)
- net M1B: now also U2.3 (IO0)
- net M2A: now also U2.17 (IO14)
- net M2B: now also U2.15 (IO12)
Changed lines of the file:
@@
 Text Label 900  1900 2    50   ~ 0
 IO2
-Text Label 900  1800 2    50   ~ 0
+Text Label 500  1700 2    50   ~ 0
 IO1
-Text Label 900  1700 2    50   ~ 0
+Text Label 500  1600 2    50   ~ 0
 IO0
 Wire Wire Line
@@
 Wire Wire Line
 	4100 5100 4550 5100
-Text Label 900  3000 2    50   ~ 0
-IO13
-Text Label 900  2900 2    50   ~ 0
+Text Label 350  2950 2    50   ~ 0
 IO12
 Text Label 900  2800 2    50   ~ 0
@@
 Text Label 10250 6250 0    50   ~ 0
 IO0
+Text Label 900  1700 2    50   ~ 0
+M1B
+Text Label 900  1800 2    50   ~ 0
+M1A
+Text Label 900  2900 2    50   ~ 0
+M2B
+Text Label 1800 3300 2    50   ~ 0
+M2A
+Text Label 900  3000 2    50   ~ 0
+IO13
 $EndSCHEMATC
